File: hardware/industrial-do4.kicad_pcb (KiCad board)
At the start: 2 copper layers, 40 x 40 mm, 24 parts, among them P1 CON-SENSOR, P2 Digital_Output, Q1 FDN5630, U1 M24C64, U2 LTV846S, U3 OPA4171AIDR, U4 DRILL, U5 DRILL, U6 DRILL, U7 DRILL

Commit message: Add 3d information (tbc)
Parts:
- C1: footprint 0603 -> kicad-libraries:C0603
- C2: footprint 0805 -> kicad-libraries:C0805
- C3: footprint ELKO_83 -> kicad-libraries:ELKO_83
- D1: footprint MiniMelf -> kicad-libraries:MiniMelf
- Fiducial_Mark (x2): footprint Fiducial_Mark -> kicad-libraries:Fiducial_Mark
- G***: footprint Logo_31x31 -> kicad-libraries:Logo_31x31
- P1: footprint CON-SENSOR -> kicad-libraries:CON-SENSOR
- P2: value Digital_Output -> Digital Output; footprint OQ_8P -> kicad-libraries:OQ_8P
- Q1: footprint SOT23GDS -> kicad-libraries:SOT23GDS
- R1: footprint 0603 -> kicad-libraries:R0603
- RP1: footprint 0603X4 -> kicad-libraries:0603X4
- RP2, RP3, RP4: footprint 1206X4 -> kicad-libraries:1206X4
- U1: footprint SOIC8 -> kicad-libraries:SOIC8
- U2: footprint OPTO-SMD16 -> kicad-libraries:OPTO-SMD16
- U3: footprint SOP14 -> kicad-libraries:SOP14
- U4, U5, U6, U7: footprint DRILL_NP -> kicad-libraries:DRILL_NP
- VAL: footprint WEEE_7mm -> kicad-libraries:WEEE_7mm
- VAL: footprint CE_5mm -> kicad-libraries:CE_5mm
Connections:
- P1 pad 1: (no net) -> Net-(P1-Pad1)
- U1 pad 7: (no net) -> Net-(U1-Pad7)
